File: Schematics/SureflapMods.kicad_sch (KiCad schematic)
At the start: 28 parts, among them K1 EE2-5NU, M1 Motor_DC, Q1 BC807, Q2 BC817, Q3 BC817, Q4 BC817, Q5 BC817, Q6 BC807, Q7 AO3400A, Q8 BC817

Commit message: Finalize schematics, EspHome works.
Parts:
- removed D5: D, symbol Device:D
- added 0R, R12, R13, R14, R15, R17, R18, R19, R20, R21, R22, R23, R24, R25, R26, R27, R28: R, symbol Device:R
- added C10, C11, C12, C13, C14, C15, C16, C17, C18, C19, C20, C21, C22, C23, C3, C6, C7, C8, C9: ~, symbol Device:C
- added C4, C5: 470µF/16V, symbol Device:C_Polarized
- added D10, D4: BAV99, Package_TO_SOT_SMD:SOT-23, symbol Diode:BAV99
- added D11: BAT54C KL3, Package_TO_SOT_SMD:SOT-23, symbol Diode:BAT54C
- added D5: MMBD2004S KAE, symbol Device:D_Dual_Series_AKC
- added D6, D8: BAS21, Package_TO_SOT_SMD:SOT-23, symbol Diode:BAS21
- added D7: BZX84Cxx WH3 ??, Package_TO_SOT_SMD:SOT-23, symbol Diode:BZX84Cxx
- added D9: BZT52Bxx C5, Diode_SMD:D_SOD-123F, symbol Diode:BZT52Bxx
- added L1: Outgoing, symbol Device:L
- added L2: Incomming, symbol Device:L
- added Q10, Q15, Q9: BC817, Package_TO_SOT_SMD:SOT-23, symbol Transistor_BJT:BC817
- added Q11: FQD6N40C, Package_TO_SOT_SMD:SOT-223-3_TabPin2, symbol Transistor_FET:NDT3055L
- added Q12: BC847W 1GW, Package_TO_SOT_SMD:SOT-323_SC-70, symbol Transistor_BJT:BC847W
- added Q13: MMBT5550LT M1F, symbol Simulation_SPICE:NPN
- added Q14: DMN6140LQ N61, Package_TO_SOT_SMD:SOT-223-3_TabPin2, symbol Transistor_FET:NDT3055L
- added Q14: N5401 2L, symbol Simulation_SPICE:PNP
- added R16: ~, symbol Device:R
- added TP1, TP2, TP3: TestPoint_Small, symbol Connector:TestPoint_Small
- added U1, U2: 74AHC1G00 ?? B003, symbol 74xGxx:74AHC1G00
- added U3: 74LVC1G79 C79J, symbol 74xGxx:74LVC1G79
- added U4: 74VHC1G86 VHC, symbol 74xGxx:74AHC1G86
- added U5: Regulator AABK SOT23, Package_TO_SOT_THT:TO-92_Inline, symbol Regulator_Linear:L78L15_TO92
- added X1: ASCO, Oscillator:Oscillator_SMD_Abracon_ASCO-4Pin_1.6x1.2mm, symbol Oscillator:ASCO
- C2: value 100n -> 10n
- R1: value 22K -> 30K
- renumbered Q6 to Q5, Q5 to Q6
Connections:
- net +6V: now also C22.2, C4.1, C5.1, D4.2 (A), D9.2 (A), U5.3 (VI)
- net GND: now also C13.1, C14.1, C15.1, C16.1, C17.1, C18.1, C19.1, C20.1, C21.1, C22.1, C23.1, C3.2, C4.2, C5.2, C6.2, D4.1 (K), D7.3 (K), D8.1 (A), Q10.2 (E), Q13.3 (E), Q14.3 (S), Q15.2 (E), R13.2, R19.1, U1.3 (GND), U2.3 (GND), U3.3 (GND), U4.3 (GND), U5.1 (GND), X1.2 (GND)
- net at K1.12, Q8.3 (C): now also D4.3 (K)
- net at K1.10: now also L1.2
- net at K1.3: now also L1.1
- net at K1.4: now also C11.1, C12.1, C7.2, D5.3 (common), Q11.2 (D)
- net at K1.5: now also L2.1
- net at K1.8: now also L2.2
- net at K1.9: now also C6.1
- net Close renamed 1 br Close
- net Dir renamed 9 wt Incomming
- net Disable renamed 5 gn Block
- net Open renamed 3 or Open
- new net: C18.2, D10.1 (K), R23.2, U1.1
- new net: R26.1, R27.1, R28.1, U3.2 (C), U4.4
- new net: R25.1, TP2.1, U1.4
- new net: 0R.1, C23.2, U5.2 (VO)
- new net: Q13.1 (C), Q14.1 (C), R16.2
- new net: C9.1, D8.3 (K), Q13.2 (B), R19.2
- new net: C15.2, C16.2, U1.5 (VCC), U2.5 (VCC)
- new net: C17.2, D10.2 (A), R22.2, U2.1
- new net: D10.3 (K), R22.1, R23.1, U3.4 (Q)
- new net: D7.1 (A), D9.1 (K)
- new net: Q11.1 (G), R16.1
- new net: C10.2, C7.1, Q11.3 (S)
- new net: R24.1, TP1.1, U2.4
- new net: C10.1, C14.2
- new net: U4.2, X1.3 (OUT)
- new net: C13.2, Q14.1 (G), R20.1
- new net: Q15.1 (B), R21.1
- new net: Q15.3 (C), R20.2
- new net: C11.2, C12.2, Q14.2 (D)
- new net: Q9.3 (C), R12.1
- new net: C8.1, D6.1 (A), Q14.2 (B), R17.1
- new net: D6.3 (K), Q14.3 (E), R17.2, R18.2
- new net +3V3: 0R.2, C19.2, C20.2, C21.2, TP3.1, U3.5 (VCC), U4.5 (VCC)
- new net 7 vi SensorBarrier: C3.1, Q9.1 (B), R12.2, R13.1
Other:
- note added: "2024.04.10"
- note added: "?"
- note added: "BC807, BC817, BC847"
- note added: "CLose to relay"
- note added: "GPIO"
- note added: "H-Bridge"
- note added: "Not sure if this part is correct and complete. I miss the supply for Q11 and Q14 Somehow the circuit must get some initial supply."
- note added: "SC3"
- note added: "STM32"
- note removed: "2024.03.21"
- note removed: "BC807, BC817"
- note removed: "H Bridge"
- moved on the sheet: BT1, C1, C2, D1, D2, D3, K1, M1, Q1, Q2, Q3, Q4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
